Commit message: remove minimum inertia and retuning gains

File: sawyer_description/urdf/sawyer_base.urdf.xacro (robot description, xacro)
@@ -9,9 +9,9 @@
   <!--  In Gazebo, links with zero principal moment of inertia (ixx, iyy, izz) could lead to infinite acceleration under any finite torque application.
       http://gazebosim.org/tutorials/?tut=ros_urdf -->
-    <inertial>
+    <!-- inertial>
       <origin rpy="0 0 0" xyz="0 0 0"/>
       <mass value="0.01"/>
       <inertia ixx="0.01" ixy="0" ixz="0" iyy="0.01" iyz="0" izz="0.01"/>
-    </inertial>
+  </inertial -->
   </xacro:macro>
   <material name="black">
@@ -170,5 +170,5 @@
     <limit effort="80.0" lower="-3.0503" upper="3.0503" velocity="1.74"/>
 <xacro:if value="$(arg gazebo)">
-    <dynamics damping="15.0" friction="5.0"/>
+    <dynamics damping="5.0" friction="2.0"/>
 </xacro:if>
   </joint>
@@ -308,5 +308,5 @@
     <limit effort="40.0" lower="-3.0439" upper="3.0439" velocity="1.957"/>
  <xacro:if value="$(arg gazebo)">
-    <dynamics damping="15.0" friction="5.0"/>
+    <dynamics damping="1.0" friction="0.5"/>
 </xacro:if>
   </joint>
@@ -338,5 +338,5 @@
     <limit effort="9.0" lower="-2.9761" upper="2.9761" velocity="3.485"/>
 <xacro:if value="$(arg gazebo)">
-    <dynamics damping="6.0" friction="1.0"/>
+    <dynamics damping="1.0" friction="0.5"/>
 </xacro:if>
   </joint>
@@ -386,5 +386,5 @@
     <limit effort="9.0" lower="-2.9761" upper="2.9761" velocity="3.485"/>
 <xacro:if value="$(arg gazebo)">
-    <dynamics damping="5.5" friction="1.2"/>
+    <dynamics damping="1.0" friction="0.5"/>
 </xacro:if>
   </joint>
@@ -452,5 +452,9 @@
     </collision>
 <xacro:if value="$(arg gazebo)">
-      <xacro:gazebo_minimum_inertia />
+    <inertial>
+      <origin rpy="0 0 0" xyz="0 0 0"/>
+      <mass value="0.01"/>
+      <inertia ixx="0.01" ixy="0" ixz="0" iyy="0.01" iyz="0" izz="0.01"/>
+    </inertial>
 </xacro:if>
 <xacro:unless value="$(arg gazebo)">

Commit message: updates minimum inertia to zero

File: sawyer_description/urdf/sawyer_base.urdf.xacro (robot description, xacro)
@@ -30,9 +30,5 @@
     <color rgba="0.75294 0.75294 0.75294 1"/>
   </material>
-  <link name="base">
-<xacro:if value="$(arg gazebo)">
-    <xacro:gazebo_minimum_inertia />
-</xacro:if>
-  </link>
+  <link name="base"/>
   <link name="torso">
     <visual>
@@ -45,7 +41,4 @@
       </material>
     </visual>
-<xacro:if value="$(arg gazebo)">
-    <xacro:gazebo_minimum_inertia />
-</xacro:if>
 <xacro:unless value="$(arg gazebo)">
     <inertial>
@@ -83,7 +76,4 @@
       </geometry>
     </collision>
-<xacro:if value="$(arg gazebo)">
-    <xacro:gazebo_minimum_inertia />
-</xacro:if>
   </link>
   <joint name="controller_box_fixed" type="fixed">
@@ -338,11 +328,8 @@
     <limit effort="9.0" lower="-2.9761" upper="2.9761" velocity="3.485"/>
 <xacro:if value="$(arg gazebo)">
-    <dynamics damping="1.0" friction="0.5"/>
+    <dynamics damping="2.0" friction="1.0"/>
 </xacro:if>
   </joint>
   <link name="right_arm_itb">
-<xacro:if value="$(arg gazebo)">
-    <xacro:gazebo_minimum_inertia />
-</xacro:if>
 <xacro:unless value="$(arg gazebo)">
     <inertial>
@@ -389,9 +376,5 @@
 </xacro:if>
   </joint>
-  <link name="right_hand_camera">
-<xacro:if value="$(arg gazebo)">
-    <xacro:gazebo_minimum_inertia />
-</xacro:if>
-  </link>
+  <link name="right_hand_camera"/>
   <joint name="right_hand_camera" type="fixed">
     <origin rpy="0 1.57079632679 0" xyz="0.039552 -0.033 0.0695"/>
@@ -400,9 +383,5 @@
     <axis xyz="0 0 0"/>
   </joint>
-  <link name="right_wrist">
-<xacro:if value="$(arg gazebo)">
-    <xacro:gazebo_minimum_inertia />
-</xacro:if>
-  </link>
+  <link name="right_wrist"/>
   <joint name="right_wrist" type="fixed">
     <origin rpy="1.57079632679 0 0" xyz="0 0 0.10541"/>
@@ -453,8 +432,8 @@
 <xacro:if value="$(arg gazebo)">
     <inertial>
-      <origin rpy="0 0 0" xyz="0 0 0"/>
+      <origin rpy="0 0 0" xyz="0 0.1 0"/>
       <mass value="0.01"/>
-      <inertia ixx="0.01" ixy="0" ixz="0" iyy="0.01" iyz="0" izz="0.01"/>
-    </inertial>
+      <inertia ixx="0.01" ixy="0.01" ixz="0.01" iyy="0.01" iyz="0.01" izz="0.01"/>
+  </inertial>
 </xacro:if>
 <xacro:unless value="$(arg gazebo)">
@@ -473,7 +452,4 @@
   </joint>
   <link name="right_l1_2">
-<xacro:if value="$(arg gazebo)">
-    <xacro:gazebo_minimum_inertia />
-</xacro:if>
 <xacro:unless value="$(arg gazebo)">
     <inertial>
@@ -497,7 +473,4 @@
   </joint>
   <link name="right_l2_2">
-<xacro:if value="$(arg gazebo)">
-    <xacro:gazebo_minimum_inertia />
-</xacro:if>
 <xacro:unless value="$(arg gazebo)">
     <inertial>
@@ -521,7 +494,4 @@
   </joint>
   <link name="right_l4_2">
-<xacro:if value="$(arg gazebo)">
-    <xacro:gazebo_minimum_inertia />
-</xacro:if>
 <xacro:unless value="$(arg gazebo)">
     <inertial>
@@ -558,7 +528,4 @@
       </geometry>
     </collision>
-<xacro:if value="$(arg gazebo)">
-    <xacro:gazebo_minimum_inertia />
-</xacro:if>
 <xacro:unless value="$(arg gazebo)">
     <inertial>
@@ -574,9 +541,5 @@
     <child link="screen"/>
   </joint>
-  <link name="head_camera">
-<xacro:if value="$(arg gazebo)">
-    <xacro:gazebo_minimum_inertia />
-</xacro:if>
-  </link>
+  <link name="head_camera"/>
   <joint name="head_camera" type="fixed">
     <origin rpy="-2.1293 0 -1.57079632679" xyz="0.0228027 0 0.216572"/>

Commit message: URDF Xacro Arg Updates
New URDF Xacro args:
- Adds "static" parameter for linking Sawyer to world frame in Gazebo
- Adds "pedestal" parameter for removing Sawyer's pedestal and
  associated frames
- Removed minimum inertia macro as it is no longer needed

File: sawyer_description/urdf/sawyer_base.urdf.xacro (robot description, xacro)
@@ -2,17 +2,5 @@
 <robot name="sawyer" xmlns:xacro="http://www.ros.org/wiki/xacro">
   <xacro:arg name="gazebo" default="false"/>
-  <xacro:if value="$(arg gazebo)">
-    <!-- Gazebo Tags -->
-    <xacro:include filename="$(find sawyer_description)/urdf/sawyer_base.gazebo.xacro" />
-  </xacro:if>
-  <xacro:macro name="gazebo_minimum_inertia">
-  <!--  In Gazebo, links with zero principal moment of inertia (ixx, iyy, izz) could lead to infinite acceleration under any finite torque application.
-      http://gazebosim.org/tutorials/?tut=ros_urdf -->
-    <!-- inertial>
-      <origin rpy="0 0 0" xyz="0 0 0"/>
-      <mass value="0.01"/>
-      <inertia ixx="0.01" ixy="0" ixz="0" iyy="0.01" iyz="0" izz="0.01"/>
-  </inertial -->
-  </xacro:macro>
+  <xacro:arg name="pedestal" default="true"/>
   <material name="black">
     <color rgba="0 0 0 1"/>
@@ -49,4 +37,5 @@
 </xacro:unless>
   </link>
+<xacro:if value="$(arg pedestal)">
   <link name="pedestal">
     <visual>
@@ -89,7 +78,4 @@
       </geometry>
     </collision>
-<xacro:if value="$(arg gazebo)">
-    <xacro:gazebo_minimum_inertia />
-</xacro:if>
   </link>
   <joint name="pedestal_feet_fixed" type="fixed">
@@ -98,4 +84,15 @@
     <child link="pedestal_feet"/>
   </joint>
+  <joint name="pedestal_fixed" type="fixed">
+    <origin rpy="0 0 0" xyz="0.0 0.0 0.0"/>
+    <parent link="base"/>
+    <child link="pedestal"/>
+  </joint>
+</xacro:if>
+  <joint name="right_arm_mount" type="fixed">
+    <origin rpy="0 0 0" xyz="0.0 0.0 0.0"/>
+    <parent link="base"/>
+    <child link="right_arm_base_link"/>
+  </joint>
   <joint name="torso_t0" type="fixed">
     <origin rpy="0 0 0" xyz="0 0 0"/>
@@ -103,14 +100,4 @@
     <child link="torso"/>
   </joint>
-  <joint name="pedestal_fixed" type="fixed">
-    <origin rpy="0 0 0" xyz="0.0 0.0 0.0"/>
-    <parent link="base"/>
-    <child link="pedestal"/>
-  </joint>
-  <joint name="right_arm_mount" type="fixed">
-    <origin rpy="0 0 0" xyz="0.0 0.0 0.0"/>
-    <parent link="base"/>
-    <child link="right_arm_base_link"/>
-  </joint>
   <link name="right_arm_base_link">
     <inertial>
@@ -194,7 +181,4 @@
   </joint>
   <link name="right_torso_itb">
-<xacro:if value="$(arg gazebo)">
-    <xacro:gazebo_minimum_inertia />
-</xacro:if>
 <xacro:unless value="$(arg gazebo)">
     <inertial>
