Commit message: compatible with gazebo8 comment cameras out

File: sawyer_description/urdf/sawyer_base.gazebo.xacro (robot description, xacro)
@@ -54,5 +54,5 @@
     <provideFeedback>true</provideFeedback>
   </gazebo>
-   <joint name="head_camera_optical_joint" type="fixed">
+  <joint name="head_camera_optical_joint" type="fixed">
     <origin xyz="0 0 0" rpy="${-pi} ${-pi/2.0} ${-pi/2.0}"/>
     <parent link="head_camera"/>
@@ -105,10 +105,10 @@
     </sensor>
   </gazebo>
-  <joint name="right_hand_camera_optical_joint" type="fixed">
+  <!-- joint name="right_hand_camera_optical_joint" type="fixed">
     <origin xyz="0 0 0" rpy="${-pi} ${-pi/2.0} ${-pi/2.0}"/>
     <parent link="right_hand_camera"/>
     <child link="right_hand_camera_optical"/>
-  </joint>
-  <link name="right_hand_camera_optical"/>
+  </joint -->
+  <!-- link name="right_hand_camera_optical"/>
   <gazebo reference="right_hand_camera_optical">
     <sensor name="right_hand_camera" type="camera">
@@ -124,5 +124,5 @@
           <near>0.02</near>
           <far>10</far>
-        </clip>
+        </clip -->
         <!-- Uncomment to add image Distortion -->
         <!-- distortion>
@@ -134,8 +134,8 @@
           <center>365.734985 237.988998</center>
         </distortion -->
-      </camera>
+      <!-- /camera -->
       <!-- Uncomment to visualize image inside Gazebo -->
       <!-- visualize>true</visualize -->
-      <plugin filename="libgazebo_ros_camera.so" name="camera_controller">
+      <!-- plugin filename="libgazebo_ros_camera.so" name="camera_controller">
         <alwaysOn>true</alwaysOn>
         <updateRate>10.0</updateRate>
@@ -144,5 +144,5 @@
         <cameraInfoTopicName>/io/internal_camera/right_hand_camera/camera_info</cameraInfoTopicName>
         <frameName>right_hand_camera</frameName>
-        <focalLength>613.760435</focalLength>
+        <focalLength>613.760435</focalLength -->
         <!-- Uncomment to add image Distortion params to camera_info topic -->
         <!-- distortionK1>-0.442</distortionK1>
@@ -153,8 +153,8 @@
         <Cx>365.734985</Cx>
         <Cy>237.988998</Cy -->
-      </plugin>
+      <!-- /plugin>
     </sensor>
-  </gazebo>
-  <gazebo reference="screen">
+  </gazebo -->
+  <!--<gazebo reference="screen">
     <visual>
       <plugin name="screen_video_controller" filename="libgazebo_ros_video.so">
@@ -165,5 +165,5 @@
       </plugin>
     </visual>
-  </gazebo>
+  </gazebo>-->
   <!-- Transmissions -->
   <!-- Right Arm -->
